File: Hardware/_saved_muse.sch (KiCad schematic (older format))
At the start: 47 parts, among them P1 3.5mm_line, P2 3.5mm_line, P3 RCA, P4 RCA, P5 ATX_PWR_OK, P6 ATX_PWR_OK, P7 ATX_PWR_OK, P8 ATX_PS_ON, P9 LED_Signal, Q1 FQP30N06L, Q2 FQP30N06L, Q3 FQP30N06L, Q4 FQP30N06L, Q5 FQP30N06L, Q6 FQP30N06L, SW1 PWR_SW, U1 MSGEQ7, U2 MSGEQ7, U3 74LS595, U4 Spark_Core

Commit message: Created custom footprints and added to PCB
Setting up PCB
Parts:
- C1, C2, C3, C4, C5, C6, C7, C8: footprint (none) -> Capacitors_ThroughHole:C_Rect_L7_W2_P5
- D1: footprint (none) -> Diodes_ThroughHole:Diode_DO-41_SOD81_Horizontal_RM10
- D2: footprint (none) -> LEDs:LED-5MM
- D3, D4, D5, D6, D7, D8, P5, P6, P7, P8: footprint (none) -> Pin_Headers:Pin_Header_Straight_1x01
- P1, P2: footprint (none) -> Pin_Headers:Pin_Header_Straight_1x03
- P3, P4: footprint (none) -> Pin_Headers:Audio_RCA_Vertical
- P9: footprint (none) -> Pin_Headers:Pin_Header_Straight_1x08
- Q1, Q2, Q3, Q4, Q5, Q6: footprint (none) -> Transistors_TO-220:TO-220_Neutral123_Horizontal_LargePads
- R1, R10, R11, R2, R3, R4, R5, R6, R7, R8, R9: footprint (none) -> Resistors_ThroughHole:Resistor_Horizontal_RM10mm
- SW1: footprint (none) -> Pin_Headers:Pin_Header_Straight_1x02
- U1, U2: footprint (none) -> Housings_DIP:DIP-8_W7.62mm_LongPads
- U3: footprint (none) -> Housings_SSOP:SSOP-16_5.3x6.2mm_Pitch0.65mm
- U4: footprint (none) -> Pin_Headers:Spark_Core
Connections:
- wire segments 173 -> 151
