File: Hardware V1.0/muse.kicad_pcb (KiCad board)
At the start: 2 copper layers, 71.6 x 61.5 mm, 51 parts, among them P1 3.5mm_line, P2 3.5mm_line, P3 RCA, P4 RCA, P8 ATX_PS_ON, P9 LED_Signal, Q1 FQP30N06L, Q2 FQP30N06L, Q3 FQP30N06L, Q4 FQP30N06L, Q5 FQP30N06L, Q6 FQP30N06L, SW1 PWR_SW, U1 MSGEQ7, U2 MSGEQ7, U3 74LS595, U4 Spark_Core

Commit message: Muse v1.3
Parts:
- removed +5V: ATX_PWR, Pin_Headers:Pin_Header_Straight_1x01
- removed ?, REF** (x3): 1pin, Connect:1pin
- removed B (x2): LED_B, Pin_Headers:Pin_Header_Straight_1x01
- removed D1: 6A, Diodes_ThroughHole:Diode_DO-41_SOD81_Horizontal_RM10
- removed G (x2): LED_G, Pin_Headers:Pin_Header_Straight_1x01
- removed GND: ATX_GND, Pin_Headers:Pin_Header_Straight_1x01
- removed P4: RCA, Pin_Headers:Audio_RCA_Vertical
- removed PWR: PWR_LED, LEDs:LED-3MM
- removed PWR_OK: ATX_PWR_OK, Pin_Headers:Pin_Header_Straight_1x01
- removed R (x2): LED_R, Pin_Headers:Pin_Header_Straight_1x01
- added D2: PWR_LED, LEDs:LED-3MM, F.Cu at (142.9, 128.3)
- added D3: LED_R, Pin_Headers:Pin_Header_Straight_1x01, F.Cu at (117.7, 128.2)
- added D4: LED_R, Pin_Headers:Pin_Header_Straight_1x01, F.Cu at (101.9, 128.2)
- added D5: LED_G, Pin_Headers:Pin_Header_Straight_1x01, F.Cu at (121.5, 128.2)
- added D6: LED_G, Pin_Headers:Pin_Header_Straight_1x01, F.Cu at (105.7, 128.2)
- added D7: LED_B, Pin_Headers:Pin_Header_Straight_1x01, F.Cu at (125.3, 128.2)
- added D8: LED_B, Pin_Headers:Pin_Header_Straight_1x01, F.Cu at (109.5, 128.2)
- added P5: ATX_PWR_OK, Pin_Headers:Pin_Header_Straight_1x01, F.Cu at (151.8, 121.9)
- added P6: ATX_PWR, Pin_Headers:Pin_Header_Straight_1x01, F.Cu at (151.8, 113.0)
- added P7: ATX_GND, Pin_Headers:Pin_Header_Straight_1x01, F.Cu at (136.5, 141.6)
- P3: footprint Pin_Headers:Audio_RCA_Vertical -> muselib:Audio_RCA_Vertical
- moved P3 0.21 mm to (83.7, 92.2)
Connections:
- P3 pad 1: GND -> (no net)
- P3 pad 2: /audio_l -> (no net)
- P3 pad 3: /audio_r -> (no net)
- U3 pad 16: (no net) -> VCC
- U3 pad 6: (no net) -> Net-(U3-Pad6)
- U3 pad 7: (no net) -> Net-(U3-Pad7)
- U3 pad 9: (no net) -> Net-(U3-Pad9)
- U4 pad 10: (no net) -> /PS_ON
- U4 pad 22: (no net) -> Net-(U4-Pad22)
- U4 pad 23: (no net) -> Net-(U4-Pad23)
- U4 pad 24: (no net) -> Net-(U4-Pad24)
- U4 pad 3: (no net) -> Net-(U4-Pad3)
- U4 pad 4: (no net) -> Net-(U4-Pad4)
Routing:
- removed copper zone on B.Cu, net GND
