File: Hardware V1.2/muse.sch (KiCad schematic (older format))
At the start: 55 parts, among them P1 3.5mm_line, P2 3.5mm_line, P3 RCA, P4 RCA, P5 ATX_PWR_OK, P6 ATX_PWR, P7 ATX_GND, P8 ATX_PS_ON, P9 LED_Signal, Q1 FQP30N06L, Q2 FQP30N06L, Q3 FQP30N06L, Q4 FQP30N06L, Q5 FQP30N06L, Q6 FQP30N06L, U1 MSGEQ7, U2 MSGEQ7, U3 74LS595, U4 Spark_Core

Commit message: Muse v1.3
Parts:
- C1, C10, C2, C3, C4, C5, C6, C7, C8, C9: symbol C-RESCUE-muse -> muse-rescue:C-RESCUE-muse
- D2, D3, D4, D5, D6, D7, D8: symbol LED-RESCUE-muse -> muse-rescue:LED-RESCUE-muse
- P1, P2: symbol CONN_01X03 -> muse-rescue:CONN_01X03
- P3, P4: symbol RCA_Stero_Jack -> muse-rescue:RCA_Stero_Jack
- P5, P6, P7, P8: symbol CONN_01X01 -> muse-rescue:CONN_01X01
- P9: symbol CONN_01X08 -> muse-rescue:CONN_01X08
- Q1, Q2, Q3, Q4, Q5, Q6: symbol Q_NMOS_GDS -> Device:Q_NMOS_GDS
- R1, R10, R11, R2, R3, R4, R5, R6, R7, R8, R9: symbol R-RESCUE-muse -> muse-rescue:R-RESCUE-muse
- R? (x8): symbol R -> muse-rescue:R
- U1, U2: symbol MSGEQ7 -> muse-rescue:MSGEQ7
- U3: symbol 74LS595 -> muse-rescue:74LS595
- U4: symbol Spark_Core -> muse-rescue:Spark_Core
Connections:
- wire segments 163 -> 187
