File: Hardware V1.3/muse.sch (KiCad schematic (older format))
At the start: 49 parts, among them CON1 RCA_conn_x2, CON2 3.5mm_conn, J1 ATX-24, J10 LED_7, J11 LED_8, J12 LED_9, J2 AUX, J3 LED_0, J4 LED_1, J5 LED_2, J6 LED_3, J7 LED_4, J8 LED_5, J9 LED_6, SW1 MCU_RST, U1 MSGEQ7, U2 MSGEQ7, U3 Photon, U4 GTL2010

Commit message: Muse v1.3
Connections:
- net +5V: now also RN2.1 (common)
- net at C9.1, R7.2, U4.23 (DREF)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: no longer RN2.1 (common)
Changed lines of the file:
@@
 	1    0    0    -1
 $EndComp
-Wire Wire Line
-	11050 1550 11400 1550
 $Comp
 L Device:R_Pack05_SIP RN3
@@
 	1    0    0    -1
 $EndComp
+$Comp
+L muse-rescue:+5V #PWR?
+U 1 1 60B29207
+P 11400 1000
+F 0 "#PWR?" H 11400 1090 20  0001 C CNN
+F 1 "+5V" H 11396 1128 30  0000 C CNN
+F 2 "" H 11400 1000 60  0000 C CNN
+F 3 "" H 11400 1000 60  0000 C CNN
+	1    11400 1000
+	1    0    0    -1
+$EndComp
+Wire Wire Line
+	11400 1000 11400 1550
 Wire Bus Line
 	7700 7800 7700 10700
